Commit message: added ultrasonic lib

File: minesweeper_ws/src/minesweeper_continuous/urdf/minesweeper_continuous.urdf (robot description, URDF)
Before this commit: robot minesweeper_continuous, 6 links, 5 joints
Joints:
- joint lwheel_bot_joint: axis 1 0 0 -> 0 0 1
- joint rwheel_bot_joint: axis 1 0 0 -> 0 0 1
- joint rwheel_top_joint: axis 1 0 0 -> 0 0 1
